Commit message: Port humble fixes to jazzy
- Fix LD250 lidar link name (laser_frame -> lidar_link) and rotation (180 -> 3.14 rad)
- Remove unused laser_frame xacro arg
- Remove static base_link -> lidar_link TF from nav2 launch (now provided by URDF)
- Default nav2 map to warehouse_with_conveyer; rename warehouse_01 -> warehouse
- Set AMR driver cmd_vel_topic to /amr/cmd_vel (fed by handsolo_filter)
- Add xhost step to README docker instructions
- Update compile workflow branch triggers

Co-Authored-By: Claude Opus 5.5 <noreply@anthropic.com>

File: handsolo_description/xacro/ld250.urdf.xacro (robot description, xacro)
@@ -3,5 +3,5 @@
   <!--
     Updated to match LD250.urdf:
-    - Adds laser_frame link
+    - Adds lidar_link
     - Adds base_link_to_laser_frame fixed joint at xyz="0.45 0 0.195"
     - Keeps main_body mesh, inertial, and fixed joints
@@ -42,5 +42,5 @@
     </joint>
     <!-- Laser frame -->
-    <link name="${prefix}laser_frame">
+    <link name="${prefix}lidar_link">
     </link>
     <!-- Base to laser frame fixed joint (matches LD250.urdf) -->
@@ -48,5 +48,5 @@
       <parent link="${prefix}base_link"/>
       <child link="${prefix}lidar_link"/>
-      <origin xyz="0.45 0 0.195" rpy="180 0 0"/>
+      <origin xyz="0.45 0 0.195" rpy="3.14 0 0"/>
     </joint>
     <!-- Optional mounting to an external parent -->

File: handsolo_description/xacro/ld250_tm12x.urdf.xacro (robot description, xacro)
@@ -6,5 +6,4 @@
   <xacro:arg name="base_prefix" default="virtual_hand_solo/"/>
   <xacro:arg name="arm_color" default="none"/>
-  <xacro:arg name="laser_frame" default="lidar_link"/>
   <xacro:arg name="trans_hw_iface" default="hardware_interface/PositionJointInterface"/>
   <xacro:arg name="arm_base_link" default="base_link"/>
