Commit message: Update MoveIt RViz, controlbox mesh and devcontainer
- MoveIt RViz: full handsolo link list, virtual_hand_solo/odom fixed frame,
  TF display and updated view (from humble)
- Use moma_description controlbox_ld250 macro (STL) instead of the removed
  LD250.obj
- Devcontainer clones omron_amr main so handsolo-ld250.yaml overrides apply

Co-Authored-By: Claude Opus 5.5 <noreply@anthropic.com>

File: handsolo_description/xacro/ld250_tm12x.urdf.xacro (robot description, xacro)
@@ -94,25 +94,6 @@
   <!--             TM12x Control box related configuration             -->
   <!-- =============================================================== -->
-  <link name="controlbox">
-    <visual>
-      <origin rpy="0 0 3.141582654" xyz="0 0 0"/>
-      <geometry>
-        <mesh filename="package://$(arg controlbox_mesh_pkg)/meshes/controlbox/LD250.obj"/>
-      </geometry>
-      <material name="controlbox_white">
-        <color rgba="1 1 1 1"/>
-      </material>
-    </visual>
-    <collision>
-      <origin rpy="0 0 3.141592654" xyz="0 0 0"/>
-      <geometry>
-        <mesh filename="package://$(arg controlbox_mesh_pkg)/meshes/controlbox/LD250.obj"/>
-      </geometry>
-    </collision>
-    <inertial>
-      <mass value="4.07"/>
-      <inertia ixx="0.426" ixy="0.0" ixz="0.0" iyy="0.496" iyz="0.0" izz="0.91"/>
-    </inertial>
-  </link>
+  <xacro:include filename="$(find moma_description)/xacro/controlbox_ld250.urdf.xacro"/>
+  <xacro:controlbox_ld250 mesh_pkg="$(arg controlbox_mesh_pkg)" link_name="controlbox"/>
   <!-- =============================================================== -->
   <!--                Joint Connection configuration                   -->
